File: Adamon/atmega.sch (EAGLE design)
At the start: 13 parts, among them IC1 5V, U1 ATMEGA328P_PDIP_EZ, Y1 16 MHZ

Commit message: updated schematic
Parts:
- added JP1: M02JST-PTH-VERT, SparkFun-Connectors:M02JST-PTH-VERT
Changed lines of the file:
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@@
 <part name="S1" library="SparkFun-Electromechanical" deviceset="TAC_SWITCH" device="SMD" value="RESET"/>
 <part name="U1" library="SparkFun-DigitalIC" deviceset="ATMEGA328P_PDIP_EZ" device=""/>
+<part name="JP1" library="SparkFun-Connectors" deviceset="M02" device="JST-PTH-VERT"/>
 </parts>
 <sheets>
@@
 <instance part="S1" gate="S" x="48.26" y="50.8"/>
 <instance part="U1" gate="G$1" x="81.28" y="33.02"/>
+<instance part="JP1" gate="G$1" x="30.48" y="71.12"/>
 </instances>
 <busses>
