File: Adamon/adamonv2.brd (EAGLE design)
At the start: 44.1 x 80 mm, 37 parts, among them IC1 5V, T1 BC337, U1 ATMEGA328P_PDIP_EZ, Y1 16 MHZ

Commit message: awh yeah
Connections:
- removed net N$3: C4.1, IC1.OUT
- net VCC: now also C4.1, IC1.OUT
Routing:
- net VCC: track 133.6 -> 141.6 mm
- net N$3: track 8.04 -> 0.00 mm
Changed lines of the file:
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@@
 <contactref element="BATTERY" pad="1"/>
-</signal>
-<signal name="N$3">
-<contactref element="IC1" pad="OUT"/>
-<contactref element="C4" pad="1"/>
-<wire x1="33.02" y1="58.42" x2="26.67" y2="58.42" width="0.254" layer="1"/>
-<wire x1="33.02" y1="59.69" x2="33.02" y2="58.42" width="0.254" layer="1"/>
-<wire x1="26.67" y1="58.42" x2="26.67" y2="58.84" width="0.254" layer="1"/>
 </signal>
 <signal name="VCC">
@@
 <wire x1="20.32" y1="49.53" x2="20.32" y2="25.4" width="0.254" layer="16"/>
 <wire x1="16.51" y1="21.59" x2="16.129" y2="21.59" width="0.254" layer="16"/>
+<contactref element="IC1" pad="OUT"/>
+<contactref element="C4" pad="1"/>
+<wire x1="33.02" y1="58.42" x2="26.67" y2="58.42" width="0.254" layer="1"/>
+<wire x1="33.02" y1="59.69" x2="33.02" y2="58.42" width="0.254" layer="1"/>
+<wire x1="26.67" y1="58.42" x2="26.67" y2="58.84" width="0.254" layer="1"/>
+<wire x1="24.13" y1="53.34" x2="26.67" y2="58.42" width="0" layer="19" extent="1-1"/>
 </signal>
 <signal name="N$4">
