File: Adamon/tiny84standalone.brd (EAGLE design)
At the start: 100 x 80 mm, 31 parts

Commit message: update tiny84
Parts:
- removed R7: 220, resistor:R0805
- removed TESTLED: GREEN, led:CHIPLED_0805
- R6: value 220 -> 330
- moved C2 161.3 mm to (48.3, 67.3)
- moved C1 155.1 mm to (41.9, 77.5)
- moved BUTTON4 137.6 mm to (36.8, 59.7)
- moved BUTTON3 120.4 mm to (26.7, 59.7)
- moved BUZZER 108.7 mm to (57.1, 72.4), turned to 180 degrees
- moved R13 104.6 mm to (66.0, 76.2), turned to 180 degrees
- moved BUTTON2 103.9 mm to (16.5, 59.7)
- moved PWRLED 98.0 mm to (61.0, 66.0), turned to 90 degrees
- moved LED4 96.1 mm to (36.8, 73.7)
- moved LED3 91.4 mm to (26.7, 73.7)
- moved BATTERY 89.8 mm to (49.5, 77.5), turned to 180 degrees
- moved S1 86.7 mm to (58.4, 59.7)
- moved GAMEMD 85.9 mm to (48.3, 59.7), turned to 90 degrees
- moved R10 84.1 mm to (19.1, 67.3), turned to 90 degrees
- moved R15 79.0 mm to (29.2, 67.3), turned to 90 degrees
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Connections:
- removed net N$7: ATTINY84.13, TESTLED.C
- removed net N$8: R7.1, TESTLED.A
- net GND: no longer R7.2
Other:
- board size 100 x 80 mm -> 75.9 x 31.7 mm

Commit message: awh yeah
Parts:
- removed S1: RESET, SparkFun-Electromechanical:TACTILE_SWITCH_SMD
- moved R3 72.7 mm to (44.5, 12.7)
- moved R2 65.9 mm to (44.5, 8.89), turned to 0 degrees
- moved BATTERY 65.7 mm to (6.35, 27.9), turned to 0 degrees
- moved R6 65.1 mm to (44.5, 16.5), turned to 180 degrees
- moved R13 64.5 mm to (27.9, 24.1), turned to 0 degrees
- moved PWRLED 63.2 mm to (44.5, 5.08), turned to 270 degrees
- moved C2 62.0 mm to (6.35, 21.6)
- moved LED1 59.7 mm to (6.35, 14.0)
- moved LED2 59.7 mm to (16.5, 14.0)
- moved LED3 59.7 mm to (26.7, 14.0)
- moved LED4 59.7 mm to (36.8, 14.0)
- moved R16 57.6 mm to (52.1, 29.2), turned to 180 degrees
- moved BUZZER 55.9 mm to (54.6, 16.5)
- moved R1 55.1 mm to (17.8, 24.1)
- moved GAMEMD 55.0 mm to (54.6, 5.08), turned to 270 degrees
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Connections:
- net GND: no longer S1.2
- net N$5: no longer S1.4
Routing:
- net N$9: track 0.00 -> 60.9 mm, vias 0 -> 2
- net N$32: track 0.00 -> 58.1 mm, vias 0 -> 1
- net VCC: track 0.00 -> 51.5 mm, vias 0 -> 2
- net N$13: track 0.00 -> 49.5 mm, vias 0 -> 1
- net N$17: track 0.00 -> 46.8 mm
- net N$20: track 0.00 -> 43.5 mm, vias 0 -> 2
- net N$12: track 0.00 -> 40.8 mm, vias 0 -> 1
- net N$18: track 0.00 -> 37.4 mm
- net N$10: track 0.00 -> 31.7 mm, vias 0 -> 2
- net N$5: track 0.00 -> 31.5 mm, vias 0 -> 1
- net N$14: track 0.00 -> 30.9 mm
- net N$35: track 0.00 -> 27.6 mm
- net N$21: track 0.00 -> 25.8 mm
- net N$22: track 0.00 -> 21.3 mm
- net N$33: track 0.00 -> 19.2 mm, vias 0 -> 2
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- added copper zone on layer 1, net GND
- added copper zone on layer 16, net GND
Other:
- board size 75.9 x 31.7 mm -> 61.9 x 31.7 mm

Commit message: better schematic
Parts:
- removed C1: 220nF, resistor:C0805
- removed R1: 10k, resistor:R0805
- removed R10, R11, R12, R2, R3, R9: 10k, rcl:R0805
- moved R6 20.1 mm to (27.9, 27.9), turned to 90 degrees
- moved R15 15.5 mm to (27.9, 21.6), turned to 270 degrees
- moved PWRLED 11.4 mm to (44.5, 16.5)
- moved R13 10.9 mm to (17.8, 27.9), turned to 270 degrees
- moved R8 10.2 mm to (12.7, 27.9), turned to 270 degrees
- moved R14 5.24 mm to (22.9, 27.9), turned to 270 degrees
- moved R16 4.02 mm to (55.9, 27.9)
Connections:
- removed net N$12: ATTINY84.6, R14.1
- removed net N$19: ATTINY84.8, R3.2
- removed net N$20: BUTTON4.4, R11.1, R12.2
- removed net N$21: ATTINY84.9, R2.2
- removed net N$22: ATTINY84.12, C1.1
- removed net N$32: LED4.K, R15.2
- removed net N$33: LED3.K, R14.2
- removed net N$35: LED2.K, R13.2
- removed net N$37: LED1.K, R8.2
- new net N$2: PWRLED.A, R6.1
- new net N$3: LED1.A, R8.2
- new net N$7: LED3.A, R14.2
- new net N$8: LED4.A, R15.2
- net GND: now also BUTTON1.1, BUTTON2.1, BUTTON3.1, BUTTON4.1, C2.2, LED1.K, LED2.K, LED3.K, LED4.K, PWRLED.C; no longer BUTTON1.2, BUTTON2.2, BUTTON3.2, BUTTON4.2, C2.1, LED1.A, LED2.A, LED3.A, LED4.A, PWRLED.A
- net N$10: now also GAMEMD.1; no longer R8.1
- net N$11: now also GAMEMD.2; no longer R13.1
- net N$13: now also ATTINY84.8, BUTTON3.3; no longer ATTINY84.7, R15.1
- net N$14: now also ATTINY84.9, BUTTON4.3; no longer BUTTON1.4, R9.2
- net N$15: now also ATTINY84.10, R8.1; no longer GAMEMD.1, R3.1
- net N$16: now also ATTINY84.11, R13.1; no longer GAMEMD.2, R2.1
- net N$17: now also ATTINY84.12, R14.1; no longer BUTTON2.4, R10.2, R9.1
- net N$18: now also ATTINY84.13, R15.1; no longer BUTTON3.4, R10.1, R11.2
- net N$4: now also LED2.A, R13.2; no longer PWRLED.C, R6.1
- net N$5: now also ATTINY84.6, BUTTON1.3; no longer ATTINY84.4, R1.1
- net N$9: now also ATTINY84.7, BUTTON2.3; no longer C1.2, R12.1
- net VCC: now also ATTINY84.4, C2.1; no longer C2.2, R1.2
Routing:
- net N$32: track 58.1 -> 0.00 mm, vias 1 -> 0
- net N$5: track 31.5 -> 80.5 mm, vias 1 -> 0
- net N$20: track 43.5 -> 0.00 mm, vias 2 -> 0
- net N$12: track 40.8 -> 0.00 mm, vias 1 -> 0
- net N$35: track 27.6 -> 0.00 mm
- net N$17: track 46.8 -> 19.7 mm, vias 0 -> 1
- net N$21: track 25.8 -> 0.00 mm
- net N$14: track 30.9 -> 56.3 mm
- net N$18: track 37.4 -> 12.3 mm
- net N$2: track 0.00 -> 23.1 mm, vias 0 -> 2
- net N$15: track 11.3 -> 33.1 mm
- net N$22: track 21.3 -> 0.00 mm
- net N$33: track 19.2 -> 0.00 mm, vias 2 -> 0
- net N$3: track 0.00 -> 17.7 mm
- net N$19: track 16.6 -> 0.00 mm, vias 1 -> 0
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