File: Adamon/tiny84standalone.sch (EAGLE design)
At the start: 31 parts

Commit message: update tiny84
Parts:
- removed R7: 220, resistor:R-US_R0805
- removed TESTLED: GREEN, led:LEDCHIPLED_0805
- R6: value 220 -> 330
Connections:
- removed net N$7: ATTINY84.(PCINT0/AREF/ADC0)PA0, TESTLED.C
- removed net N$8: R7.1, TESTLED.A
- net GND: no longer R7.2
Changed lines of the file:
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@@
 <parts>
 <part name="PWRLED" library="led" deviceset="LED" device="CHIPLED_0805" value="RED"/>
-<part name="TESTLED" library="led" deviceset="LED" device="CHIPLED_0805" value="GREEN"/>
-<part name="R6" library="resistor" deviceset="R-US_" device="R0805" value="220"/>
-<part name="R7" library="resistor" deviceset="R-US_" device="R0805" value="220"/>
+<part name="R6" library="resistor" deviceset="R-US_" device="R0805" value="330"/>
 <part name="R1" library="resistor" deviceset="R-US_" device="R0805" value="10k"/>
 <part name="S1" library="SparkFun-Electromechanical" deviceset="TAC_SWITCH" device="SMD" value="RESET"/>
@@
 <part name="SUPPLY4" library="supply2" deviceset="GND" device=""/>
 <part name="SUPPLY7" library="supply2" deviceset="GND" device=""/>
-<part name="SUPPLY8" library="supply2" deviceset="GND" device=""/>
 <part name="SUPPLY3" library="supply2" deviceset="GND" device=""/>
 <part name="P+1" library="supply1" deviceset="VCC" device=""/>
@@
 <instances>
 <instance part="PWRLED" gate="G$1" x="45.72" y="132.08" rot="R90"/>
-<instance part="TESTLED" gate="G$1" x="38.1" y="58.42" rot="R90"/>
 <instance part="R6" gate="G$1" x="58.42" y="132.08"/>
-<instance part="R7" gate="G$1" x="25.4" y="58.42" rot="R180"/>
 <instance part="R1" gate="G$1" x="33.02" y="106.68" rot="R180"/>
 <instance part="S1" gate="S" x="35.56" y="116.84"/>
@@
 <instance part="SUPPLY4" gate="GND" x="10.16" y="68.58" rot="R270"/>
 <instance part="SUPPLY7" gate="GND" x="25.4" y="114.3" rot="R270"/>
-<instance part="SUPPLY8" gate="GND" x="15.24" y="58.42" rot="R270"/>
 <instance part="SUPPLY3" gate="GND" x="35.56" y="132.08" rot="R270"/>
 <instance part="P+1" gate="VCC" x="68.58" y="132.08" rot="R270"/>
@@
 </segment>
 <segment>
-<pinref part="R7" gate="G$1" pin="2"/>
-<pinref part="SUPPLY8" gate="GND" pin="GND"/>
-<wire x1="20.32" y1="58.42" x2="17.78" y2="58.42" width="0.1524" layer="91"/>
-</segment>
-<segment>
 <pinref part="PWRLED" gate="G$1" pin="A"/>
 <wire x1="38.1" y1="132.08" x2="43.18" y2="132.08" width="0.1524" layer="91"/>
@@
 </segment>
 </net>
-<net name="N$7" class="0">
-<segment>
-<pinref part="TESTLED" gate="G$1" pin="C"/>
-<wire x1="43.18" y1="58.42" x2="66.04" y2="58.42" width="0.1524" layer="91"/>
-<wire x1="66.04" y1="58.42" x2="66.04" y2="68.58" width="0.1524" layer="91"/>
-<pinref part="ATTINY84" gate="G$1" pin="(PCINT0/AREF/ADC0)PA0"/>
-</segment>
-</net>
-<net name="N$8" class="0">
-<segment>
-<pinref part="TESTLED" gate="G$1" pin="A"/>
-<pinref part="R7" gate="G$1" pin="1"/>
-<wire x1="35.56" y1="58.42" x2="30.48" y2="58.42" width="0.1524" layer="91"/>
-</segment>
-</net>

Commit message: awh yeah
Parts:
- removed S1: RESET, SparkFun-Electromechanical:TAC_SWITCHSMD
Connections:
- net GND: no longer S1.2
- net N$5: no longer S1.4
Other:
- moved on the sheet: PWRLED, R6
Changed lines of the file:
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@@
 <part name="R6" library="resistor" deviceset="R-US_" device="R0805" value="330"/>
 <part name="R1" library="resistor" deviceset="R-US_" device="R0805" value="10k"/>
-<part name="S1" library="SparkFun-Electromechanical" deviceset="TAC_SWITCH" device="SMD" value="RESET"/>
 <part name="BATTERY" library="SparkFun-Connectors" deviceset="M02" device="JST-PTH-VERT"/>
 <part name="P+2" library="supply1" deviceset="VCC" device=""/>
 <part name="P+3" library="supply1" deviceset="VCC" device=""/>
 <part name="SUPPLY4" library="supply2" deviceset="GND" device=""/>
-<part name="SUPPLY7" library="supply2" deviceset="GND" device=""/>
 <part name="SUPPLY3" library="supply2" deviceset="GND" device=""/>
 <part name="P+1" library="supply1" deviceset="VCC" device=""/>
@@
 </plain>
 <instances>
-<instance part="PWRLED" gate="G$1" x="45.72" y="132.08" rot="R90"/>
-<instance part="R6" gate="G$1" x="58.42" y="132.08"/>
+<instance part="PWRLED" gate="G$1" x="40.64" y="114.3" rot="R90"/>
+<instance part="R6" gate="G$1" x="53.34" y="114.3"/>
 <instance part="R1" gate="G$1" x="33.02" y="106.68" rot="R180"/>
-<instance part="S1" gate="S" x="35.56" y="116.84"/>
 <instance part="BATTERY" gate="G$1" x="2.54" y="137.16" rot="MR180"/>
 <instance part="P+2" gate="VCC" x="20.32" y="121.92"/>
 <instance part="P+3" gate="VCC" x="7.62" y="99.06" rot="R90"/>
 <instance part="SUPPLY4" gate="GND" x="10.16" y="68.58" rot="R270"/>
-<instance part="SUPPLY7" gate="GND" x="25.4" y="114.3" rot="R270"/>
-<instance part="SUPPLY3" gate="GND" x="35.56" y="132.08" rot="R270"/>
-<instance part="P+1" gate="VCC" x="68.58" y="132.08" rot="R270"/>
+<instance part="SUPPLY3" gate="GND" x="30.48" y="114.3" rot="R270"/>
+<instance part="P+1" gate="VCC" x="63.5" y="114.3" rot="R270"/>
 <instance part="R12" gate="G$1" x="66.04" y="50.8" rot="MR0"/>
 <instance part="LED4" gate="G$1" x="106.68" y="68.58" rot="R270"/>
@@
 </segment>
 <segment>
-<pinref part="SUPPLY7" gate="GND" pin="GND"/>
-<pinref part="S1" gate="S" pin="2"/>
-<wire x1="27.94" y1="114.3" x2="30.48" y2="114.3" width="0.1524" layer="91"/>
-</segment>
-<segment>
 <pinref part="PWRLED" gate="G$1" pin="A"/>
-<wire x1="38.1" y1="132.08" x2="43.18" y2="132.08" width="0.1524" layer="91"/>
+<wire x1="33.02" y1="114.3" x2="38.1" y2="114.3" width="0.1524" layer="91"/>
 <pinref part="SUPPLY3" gate="GND" pin="GND"/>
 </segment>
@@
 <segment>
 <pinref part="R6" gate="G$1" pin="2"/>
-<wire x1="63.5" y1="132.08" x2="66.04" y2="132.08" width="0.1524" layer="91"/>
+<wire x1="58.42" y1="114.3" x2="60.96" y2="114.3" width="0.1524" layer="91"/>
 <pinref part="P+1" gate="VCC" pin="VCC"/>
 </segment>
@@
 <pinref part="PWRLED" gate="G$1" pin="C"/>
 <pinref part="R6" gate="G$1" pin="1"/>
-<wire x1="50.8" y1="132.08" x2="53.34" y2="132.08" width="0.1524" layer="91"/>
+<wire x1="45.72" y1="114.3" x2="48.26" y2="114.3" width="0.1524" layer="91"/>
 </segment>
 </net>
 <net name="N$5" class="0">
 <segment>
-<pinref part="S1" gate="S" pin="4"/>
-<wire x1="40.64" y1="114.3" x2="45.72" y2="114.3" width="0.1524" layer="91"/>
 <pinref part="R1" gate="G$1" pin="1"/>
-<wire x1="38.1" y1="106.68" x2="45.72" y2="106.68" width="0.1524" layer="91"/>
-<wire x1="45.72" y1="106.68" x2="71.12" y2="106.68" width="0.1524" layer="91"/>
+<wire x1="38.1" y1="106.68" x2="71.12" y2="106.68" width="0.1524" layer="91"/>
 <wire x1="71.12" y1="106.68" x2="71.12" y2="99.06" width="0.1524" layer="91"/>
 <pinref part="ATTINY84" gate="G$1" pin="(PCINT11/~RESET/DW)PB3"/>
 <wire x1="71.12" y1="99.06" x2="66.04" y2="99.06" width="0.1524" layer="91"/>
-<wire x1="45.72" y1="114.3" x2="45.72" y2="106.68" width="0.1524" layer="91"/>
-<junction x="45.72" y="106.68"/>
-</segment>
-</net>
+</segment>
+</net>

Commit message: better schematic
Parts:
- removed C1: 220nF, resistor:C-USC0805
- removed R1: 10k, resistor:R-US_R0805
- removed R10, R11, R12, R2, R3, R9: 10k, rcl:R-US_R0805
Connections:
- removed net N$12: ATTINY84.(PCINT7/ICP/OC0B/ADC7)PA7, R14.1
- removed net N$19: ATTINY84.(PCINT5/OC1B/MISO/DO/ADC5)PA5, R3.2
- removed net N$20: BUTTON4.4, R11.1, R12.2
- removed net N$21: ATTINY84.(PCINT4/T1/SCL/USCK/ADC4)PA4, R2.2
- removed net N$22: ATTINY84.(PCINT1/AIN0/ADC1)PA1, C1.1
- removed net N$32: LED4.C, R15.2
- removed net N$33: LED3.C, R14.2
- removed net N$35: LED2.C, R13.2
- removed net N$37: LED1.C, R8.2
- new net N$2: PWRLED.A, R6.1
- new net N$3: LED1.A, R8.2
- new net N$7: LED3.A, R14.2
- new net N$8: LED4.A, R15.2
- net GND: now also BUTTON1.1, BUTTON2.1, BUTTON3.1, BUTTON4.1, C2.-, LED1.C, LED2.C, LED3.C, LED4.C, PWRLED.C; no longer BUTTON1.2, BUTTON2.2, BUTTON3.2, BUTTON4.2, C2.+, LED1.A, LED2.A, LED3.A, LED4.A, PWRLED.A
- net N$10: now also GAMEMD.1; no longer R8.1
- net N$11: now also GAMEMD.2; no longer R13.1
- net N$13: now also ATTINY84.(PCINT5/OC1B/MISO/DO/ADC5)PA5, BUTTON3.3; no longer ATTINY84.(PCINT6/OC1A/SDA/MOSI/ADC6)PA6, R15.1
- net N$14: now also ATTINY84.(PCINT4/T1/SCL/USCK/ADC4)PA4, BUTTON4.3; no longer BUTTON1.4, R9.2
- net N$15: now also ATTINY84.(PCINT3/T0/ADC3)PA3, R8.1; no longer GAMEMD.1, R3.1
- net N$16: now also ATTINY84.(PCINT2/AIN1/ADC2)PA2, R13.1; no longer GAMEMD.2, R2.1
- net N$17: now also ATTINY84.(PCINT1/AIN0/ADC1)PA1, R14.1; no longer BUTTON2.4, R10.2, R9.1
- net N$18: now also ATTINY84.(PCINT0/AREF/ADC0)PA0, R15.1; no longer BUTTON3.4, R10.1, R11.2
- net N$4: now also LED2.A, R13.2; no longer PWRLED.C, R6.1
- net N$5: now also ATTINY84.(PCINT7/ICP/OC0B/ADC7)PA7, BUTTON1.3; no longer ATTINY84.(PCINT11/~RESET/DW)PB3, R1.1
- net N$9: now also ATTINY84.(PCINT6/OC1A/SDA/MOSI/ADC6)PA6, BUTTON2.3; no longer C1.2, R12.1
- net VCC: now also ATTINY84.(PCINT11/~RESET/DW)PB3, C2.+; no longer C2.-, R1.2
Other:
- moved on the sheet: BATTERY, BUTTON1, BUTTON2, BUTTON3, BUTTON4, C2, GAMEMD, LED1, LED2, LED3, LED4, PWRLED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
